Commit message: urdf logic updated

File: src/canopyag_description/urdf/canopyag.urdf.xacro (robot description, xacro)
@@ -1,14 +1,10 @@
 <?xml version="1.0"?>
 <!--
-  canopy.ag SCARA - top-level description.
-  Build it by hand to check your edits:
+  Top level. Every number comes from config/robot_parameters.yaml, which the
+  importer regenerates from a SolidWorks export - there is nothing robot
+  specific in any of the xacro files.
+  Expand it by hand to check an edit:
     xacro canopyag.urdf.xacro sim:=false > /tmp/canopyag.urdf
     check_urdf /tmp/canopyag.urdf
-    urdf_to_graphiz /tmp/canopyag.urdf     # renders the kinematic tree to PDF
-  Args:
-    sim            true  -> gz_ros2_control plugin + Gazebo tags
-                   false -> the CAN/serial hardware interfaces
-    use_meshes     override the value in arm_parameters.yaml
-    can_interface  SocketCAN device name (ip link show)
 -->
 <robot xmlns:xacro="http://www.ros.org/wiki/xacro" name="canopyag">
@@ -16,33 +12,19 @@
   <xacro:arg name="can_interface" default="can0"/>
   <xacro:arg name="can_bitrate"   default="500000"/>
-  <xacro:arg name="use_meshes"    default=""/>
   <xacro:arg name="params_file"
-             default="$(find canopyag_description)/config/arm_parameters.yaml"/>
+             default="$(find canopyag_description)/config/robot_parameters.yaml"/>
   <xacro:arg name="controllers_file"
              default="$(find canopyag_description)/config/controllers.yaml"/>
-  <xacro:include filename="$(find canopyag_description)/urdf/common.xacro"/>
-  <xacro:include filename="$(find canopyag_description)/urdf/arm.xacro"/>
-  <xacro:include filename="$(find canopyag_description)/urdf/gripper.xacro"/>
-  <xacro:include filename="$(find canopyag_description)/urdf/canopyag.ros2_control.xacro"/>
+  <xacro:include filename="$(find canopyag_description)/urdf/macros.xacro"/>
+  <xacro:include filename="$(find canopyag_description)/urdf/ros2_control.xacro"/>
   <xacro:include filename="$(find canopyag_description)/urdf/gazebo.xacro"/>
   <xacro:property name="cfg" value="${xacro.load_yaml('$(arg params_file)')}"/>
   <xacro:property name="sim" value="$(arg sim)"/>
-  <xacro:property name="use_meshes"
-                  value="${'$(arg use_meshes)' if '$(arg use_meshes)' != '' else cfg['options']['use_meshes']}"/>
-  <!-- The column is bolted down. If the SCARA ever goes on a rail or an AMR,
-       replace this fixed joint - do not move base_link itself. -->
-  <link name="world"/>
-  <joint name="world_to_base" type="fixed">
-    <parent link="world"/>
-    <child  link="base_link"/>
-    <origin xyz="0 0 ${cfg['options']['floor_offset']}" rpy="0 0 0"/>
-  </joint>
-  <xacro:canopyag_arm cfg="${cfg}" use_meshes="${use_meshes}"/>
-  <xacro:canopyag_gripper cfg="${cfg}" use_meshes="${use_meshes}" parent="tool_link"/>
-  <xacro:canopyag_ros2_control cfg="${cfg}" sim="${sim}"
-                               can_interface="$(arg can_interface)"
-                               can_bitrate="$(arg can_bitrate)"/>
+  <xacro:build_robot cfg="${cfg}"/>
+  <xacro:build_ros2_control cfg="${cfg}" sim="${sim}"
+                            can_interface="$(arg can_interface)"
+                            can_bitrate="$(arg can_bitrate)"/>
   <xacro:if value="${sim}">
-    <xacro:canopyag_gazebo controllers_file="$(arg controllers_file)"/>
+    <xacro:build_gazebo controllers_file="$(arg controllers_file)"/>
   </xacro:if>
 </robot>

File: src/canopyag_description/urdf/gazebo.xacro (robot description, xacro)
@@ -1,19 +1,8 @@
 <?xml version="1.0"?>
 <robot xmlns:xacro="http://www.ros.org/wiki/xacro">
-  <!-- Friction/contact for the jaws, otherwise grasped fruit slides straight
-       out. mu=1.2 is deliberately high - assume rubber-faced jaws. -->
-  <xacro:macro name="jaw_surface" params="link">
-    <gazebo reference="${link}">
-      <mu1>1.2</mu1>
-      <mu2>1.2</mu2>
-      <kp>1000000.0</kp>
-      <kd>100.0</kd>
-      <minDepth>0.001</minDepth>
-    </gazebo>
-  </xacro:macro>
-  <xacro:macro name="canopyag_gazebo" params="controllers_file">
-    <!-- gz_ros2_control spawns the controller_manager INSIDE the sim process
-         so it steps in lockstep with physics. There is no separate
-         ros2_control_node when simulating - do not launch one. -->
+  <!-- gz_ros2_control hosts the controller_manager inside the sim process so
+       it steps in lockstep with physics. There is no separate
+       ros2_control_node when simulating - do not launch one. -->
+  <xacro:macro name="build_gazebo" params="controllers_file">
     <gazebo>
       <plugin filename="gz_ros2_control-system"
@@ -22,6 +11,4 @@
       </plugin>
     </gazebo>
-    <xacro:jaw_surface link="left_finger_link"/>
-    <xacro:jaw_surface link="right_finger_link"/>
   </xacro:macro>
 </robot>

Commit message: added moveit demo and updated readme

File: src/canopyag_description/urdf/canopyag.urdf.xacro (robot description, xacro)
@@ -10,4 +10,6 @@
 <robot xmlns:xacro="http://www.ros.org/wiki/xacro" name="canopyag">
   <xacro:arg name="sim"           default="true"/>
+  <!-- Only read when sim is false: mock hardware instead of the CAN bus. -->
+  <xacro:arg name="mock"          default="false"/>
   <xacro:arg name="can_interface" default="can0"/>
   <xacro:arg name="can_bitrate"   default="500000"/>
@@ -22,5 +24,5 @@
   <xacro:property name="sim" value="$(arg sim)"/>
   <xacro:build_robot cfg="${cfg}"/>
-  <xacro:build_ros2_control cfg="${cfg}" sim="${sim}"
+  <xacro:build_ros2_control cfg="${cfg}" sim="${sim}" mock="$(arg mock)"
                             can_interface="$(arg can_interface)"
                             can_bitrate="$(arg can_bitrate)"/>

File: src/canopyag_description/urdf/macros.xacro (robot description, xacro)
@@ -47,9 +47,22 @@
           <material name="${L['material']}"/>
         </visual>
+        <xacro:unless value="${'collision_box' in L}">
+          <collision>
+            <origin xyz="${L['visual_xyz'][0]} ${L['visual_xyz'][1]} ${L['visual_xyz'][2]}"
+                    rpy="${L['visual_rpy'][0]} ${L['visual_rpy'][1]} ${L['visual_rpy'][2]}"/>
+            <geometry>
+              <mesh filename="package://${M['package']}/${col_dir}/${L['mesh']}" scale="${S}"/>
+            </geometry>
+          </collision>
+        </xacro:unless>
+      </xacro:if>
+      <!-- A hand-written box replaces the mesh for collision: cheap to check,
+           and it does not change when the CAD does. -->
+      <xacro:if value="${'collision_box' in L}">
+        <xacro:property name="B" value="${L['collision_box']}"/>
         <collision>
-          <origin xyz="${L['visual_xyz'][0]} ${L['visual_xyz'][1]} ${L['visual_xyz'][2]}"
-                  rpy="${L['visual_rpy'][0]} ${L['visual_rpy'][1]} ${L['visual_rpy'][2]}"/>
+          <origin xyz="${B['xyz'][0]} ${B['xyz'][1]} ${B['xyz'][2]}" rpy="0 0 0"/>
           <geometry>
-            <mesh filename="package://${M['package']}/${col_dir}/${L['mesh']}" scale="${S}"/>
+            <box size="${B['size'][0]} ${B['size'][1]} ${B['size'][2]}"/>
           </geometry>
         </collision>

File: src/canopyag_description/urdf/ros2_control.xacro (robot description, xacro)
@@ -2,7 +2,10 @@
 <!--
   One <ros2_control> system holding every non-fixed joint from
-  robot_parameters.yaml. `sim` picks the hardware plugin and is the only
-  difference between Gazebo and the real robot - the URDF, the controllers and
-  MoveIt are identical either way.
+  robot_parameters.yaml. `sim` and `mock` pick the hardware plugin and are the
+  only difference between Gazebo, mock hardware and the real robot - the URDF,
+  the controllers and MoveIt are identical either way.
+  mock:=true uses ros2_control's mock_components/GenericSystem: every command
+  is reflected straight back as state. No physics, no hardware - what the
+  MoveIt demo runs on until the real axes exist.
 -->
 <robot xmlns:xacro="http://www.ros.org/wiki/xacro">
@@ -23,5 +26,5 @@
     </xacro:if>
   </xacro:macro>
-  <xacro:macro name="build_ros2_control" params="cfg sim can_interface can_bitrate">
+  <xacro:macro name="build_ros2_control" params="cfg sim mock can_interface can_bitrate">
     <ros2_control name="${cfg['robot']['name']}" type="system">
       <hardware>
@@ -29,5 +32,8 @@
           <plugin>gz_ros2_control/GazeboSimSystem</plugin>
         </xacro:if>
-        <xacro:unless value="${sim}">
+        <xacro:if value="${mock and not sim}">
+          <plugin>mock_components/GenericSystem</plugin>
+        </xacro:if>
+        <xacro:unless value="${sim or mock}">
           <!-- Implemented in canopyag_hardware, which does not exist yet. -->
           <plugin>canopyag_hardware/CanopyagSystem</plugin>

Commit message: added connection to CAN

File: src/canopyag_description/urdf/canopyag.urdf.xacro (robot description, xacro)
@@ -14,4 +14,7 @@
   <xacro:arg name="can_interface" default="can0"/>
   <xacro:arg name="can_bitrate"   default="500000"/>
+  <!-- Joint <-> motor mapping, only read on the real robot. -->
+  <xacro:arg name="hardware_file"
+             default="$(find canopyag_description)/config/hardware.yaml"/>
   <xacro:arg name="params_file"
              default="$(find canopyag_description)/config/robot_parameters.yaml"/>
@@ -26,5 +29,6 @@
   <xacro:build_ros2_control cfg="${cfg}" sim="${sim}" mock="$(arg mock)"
                             can_interface="$(arg can_interface)"
-                            can_bitrate="$(arg can_bitrate)"/>
+                            can_bitrate="$(arg can_bitrate)"
+                            hardware_file="$(arg hardware_file)"/>
   <xacro:if value="${sim}">
     <xacro:build_gazebo controllers_file="$(arg controllers_file)"/>

File: src/canopyag_description/urdf/ros2_control.xacro (robot description, xacro)
@@ -8,10 +8,24 @@
   is reflected straight back as state. No physics, no hardware - what the
   MoveIt demo runs on until the real axes exist.
+  Neither: canopyag_hardware/CanopyagSystem on SocketCAN. Only then is
+  config/hardware.yaml loaded, and its values become <param> tags on the
+  <hardware> and on each <joint>. Sim and mock output does not depend on it.
 -->
 <robot xmlns:xacro="http://www.ros.org/wiki/xacro">
-  <xacro:macro name="axis_each" params="names cfg">
+  <!-- One <param name="key">value</param> per entry of the dict `d`. -->
+  <xacro:macro name="param_each" params="keys d">
+    <xacro:if value="${len(keys) > 0}">
+      <param name="${keys[0]}">${d[keys[0]]}</param>
+      <xacro:param_each keys="${keys[1:]}" d="${d}"/>
+    </xacro:if>
+  </xacro:macro>
+  <!-- hw: the joints: table of hardware.yaml, or empty for sim / mock. -->
+  <xacro:macro name="axis_each" params="names cfg hw">
     <xacro:if value="${len(names) > 0}">
       <xacro:property name="J" value="${cfg['joints'][names[0]]}"/>
       <joint name="${names[0]}">
+        <xacro:if value="${names[0] in hw}">
+          <xacro:param_each keys="${list(hw[names[0]].keys())}" d="${hw[names[0]]}"/>
+        </xacro:if>
         <command_interface name="position">
           <xacro:if value="${'lower' in J['limit']}">
@@ -23,8 +37,11 @@
         <state_interface name="velocity"/>
       </joint>
-      <xacro:axis_each names="${names[1:]}" cfg="${cfg}"/>
+      <xacro:axis_each names="${names[1:]}" cfg="${cfg}" hw="${hw}"/>
     </xacro:if>
   </xacro:macro>
-  <xacro:macro name="build_ros2_control" params="cfg sim mock can_interface can_bitrate">
+  <xacro:macro name="build_ros2_control" params="cfg sim mock can_interface can_bitrate hardware_file">
+    <xacro:property name="real" value="${not (sim or mock)}"/>
+    <xacro:property name="hw_cfg"
+                    value="${xacro.load_yaml(hardware_file) if real else dict(hardware=dict(), joints=dict())}"/>
     <ros2_control name="${cfg['robot']['name']}" type="system">
       <hardware>
@@ -36,11 +53,12 @@
         </xacro:if>
         <xacro:unless value="${sim or mock}">
-          <!-- Implemented in canopyag_hardware, which does not exist yet. -->
+          <!-- src/canopyag_hardware; joint mapping in config/hardware.yaml -->
           <plugin>canopyag_hardware/CanopyagSystem</plugin>
           <param name="can_interface">${can_interface}</param>
           <param name="can_bitrate">${can_bitrate}</param>
+          <xacro:param_each keys="${list(hw_cfg['hardware'].keys())}" d="${hw_cfg['hardware']}"/>
         </xacro:unless>
       </hardware>
-      <xacro:axis_each cfg="${cfg}"
+      <xacro:axis_each cfg="${cfg}" hw="${hw_cfg['joints']}"
         names="${[n for n, J in cfg['joints'].items() if J['type'] != 'fixed']}"/>
     </ros2_control>
